File: 004-AdditiveVCO/Hardware/AdditiveVCO/AdditiveVCO.kicad_sch (KiCad schematic)
At the start: 30 parts, among them J1 VOCT_IN, J2 CV_HARM, J3 CV_HARM, J4 OUT, U1 MCP6002-xP

Commit message: Finished up AdditiveVCO project
Parts:
- C1, C2, C3, C4, C5, C6, C7, C8: footprint (none) -> Capacitor_THT:C_Rect_L7.0mm_W2.0mm_P5.00mm
- J1, J2, J4: footprint (none) -> Connector_Pin:Pin_D0.7mm_L6.5mm_W1.8mm_FlatFork
- J3: value CV_HARM -> CV_GAIN; footprint (none) -> Connector_Pin:Pin_D0.7mm_L6.5mm_W1.8mm_FlatFork
- R1, R10, R11, R12, R13, R2, R3, R4, R5, R6, R7, R8, R9: footprint (none) -> Resistor_THT:R_Axial_DIN0207_L6.3mm_D2.5mm_P10.16mm_Horizontal
- RV1, RV2, RV3: footprint (none) -> Potentiometer_THT:Potentiometer_Alpha_RD901F-40-00D_Single_Vertical
- U1: footprint (none) -> Package_DIP:DIP-8_W7.62mm
Other:
- moved on the sheet: C1, C2, C3, C4, C5, C6, J1, J2, J3, R1, R2, R3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
